Commit message: feat: robot description with new vehicle stl

File: src/isa_afa_3/src/description/robot.xacro (robot description, xacro)
@@ -1,10 +1,10 @@
 <?xml version="1.0"?>
 <robot name="robot" xmlns:xacro="http://www.ros.org/wiki/xacro">
-    <xacro:include filename="$(find isa_afa_3)/urdf/robot.gazebo" />
+    <xacro:include filename="$(find isa_afa_3)/src/description/robot.gazebo" />
     <!-- Parameters -->
     <xacro:property name="chassis_mass" value="10" />
     <!-- LINKS -->
     <!-- Link - chassis -->
-    <link name="link_chassis">
+    <link name="base_link">
         <inertial>
             <mass value="${chassis_mass}" />
@@ -13,11 +13,13 @@
         </inertial>
         <collision>
-            <geometry>
-                <mesh filename="package://isa_afa_3/meshes/chassis.stl" />
-            </geometry>
-        </collision>
-        <visual>
-            <geometry>
-                <mesh filename="package://isa_afa_3/meshes/chassis.stl" />
+            <origin xyz="0 0 0" rpy="0 0 0"/>
+            <geometry>
+                <mesh filename="package://isa_afa_3/meshes/chassis.stl"/>
+            </geometry>
+        </collision>
+        <visual>
+            <origin xyz="0 0 0" rpy="0 0 0"/>
+            <geometry>
+                <mesh filename="package://isa_afa_3/meshes/chassis.stl"/>
             </geometry>
             <material name="DarkBlue">
@@ -26,206 +28,152 @@
         </visual>
     </link>
+    <!-- Robot Footprint -->
+    <link name='base_footprint'>
+        <inertial>
+            <mass value="${chassis_mass}" />
+            <origin xyz="0 0 0.3" rpy="0 0 0" />
+            <inertia ixx="1.5417" ixy="0" ixz="0" iyy="3.467" iyz="0" izz="4.742" />
+        </inertial>
+    </link>
     <!-- Link - rear left wheel -->
-    <link name="link_rear_left_wheel">
-        <inertial>
-            <mass value="1" />
-            <origin xyz="0 0 0" rpy="0 0 0" />
-            <inertia ixx="0.002526666666667" ixy="0" ixz="0" iyy="0.002526666666667" iyz="0" izz="0.005"/>
-        </inertial>
-        <!-- Tires -->
-        <collision>
-            <origin rpy="${pi/2} 0 0" xyz="0 0.18 0" />
-            <geometry>
-                <cylinder length="0.12" radius="0.4"/>
-            </geometry>
-        </collision>
-        <visual>
-            <origin rpy="${pi/2} 0 0" xyz="0 0.18 0" />
-            <geometry>
-                <mesh filename="package://isa_afa_3/meshes/wheel.stl" />
-            </geometry>
-            <material name="Black">
-                <color rgba="0.1 0.1 0.1 1" />
-            </material>
-        </visual>
-        <!-- Axle -->
-        <collision>
-            <origin rpy="${pi/2} 0 0" xyz="0 0.06 0" />
-            <geometry>
-                <cylinder length="0.12" radius="0.08"/>
-            </geometry>
-        </collision>
-        <visual>
-            <origin rpy="${pi/2} 0 0" xyz="0 0.06 0" />
-            <geometry>
-                <cylinder length="0.12" radius="0.08"/>
-            </geometry>
-            <material name="Grey">
-                <color rgba="0.6 0.6 0.6 1" />
-            </material>
-        </visual>
-        <!-- Hubcap -->
-        <visual>
-            <origin rpy="${pi/2} 0 0" xyz="0 0.18 0" />
-            <geometry>
-                <box size="0.02 0.5 0.02" />
-            </geometry>
-            <material name="Grey">
-                <color rgba="0.6 0.6 0.6 1" />
+    <link name="rear_left_wheel_link">
+        <inertial>
+            <mass value="1" />
+            <origin xyz="0 0 0" rpy="0 0 0" />
+            <inertia ixx="0.002526666666667" ixy="0" ixz="0" iyy="0.002526666666667" iyz="0" izz="0.005"/>
+        </inertial>
+        <collision>
+            <origin xyz="0 0 0" rpy="0 0 0"/>
+            <geometry>
+                <mesh filename="package://isa_afa_3/meshes/wheel_left.stl" />
+            </geometry>
+        </collision>
+        <visual>
+            <origin xyz="0 0 0" rpy="0 0 0"/>
+            <geometry>
+                <mesh filename="package://isa_afa_3/meshes/wheel_left.stl" />
+            </geometry>
+            <material name="Black">
+                <color rgba="0.1 0.1 0.1 1" />
             </material>
         </visual>
     </link>
     <!-- Link - rear right wheel -->
-    <link name="link_rear_right_wheel">
-        <inertial>
-            <mass value="1" />
-            <origin xyz="0 0 0" rpy="0 0 0" />
-            <inertia ixx="0.002526666666667" ixy="0" ixz="0" iyy="0.002526666666667" iyz="0" izz="0.005"/>
-        </inertial>
-        <!-- Tires -->
-        <collision>
-            <origin rpy="${pi/2} 0 0" xyz="0 -0.18 0" />
-            <geometry>
-                <cylinder length="0.12" radius="0.4"/>
-            </geometry>
-        </collision>
-        <visual>
-            <origin rpy="${pi/2} 0 0" xyz="0 -0.18 0" />
-            <geometry>
-                <mesh filename="package://isa_afa_3/meshes/wheel.stl" />
-            </geometry>
-            <material name="Black">
-                <color rgba="0.1 0.1 0.1 1" />
-            </material>
-        </visual>
-        <!-- Axle -->
-        <collision>
-            <origin rpy="${pi/2} 0 0" xyz="0 -0.06 0" />
-            <geometry>
-                <cylinder length="0.12" radius="0.08"/>
-            </geometry>
-        </collision>
-        <visual>
-            <origin rpy="${pi/2} 0 0" xyz="0 -0.06 0" />
-            <geometry>
-                <cylinder length="0.12" radius="0.08"/>
-            </geometry>
-            <material name="Grey">
-                <color rgba="0.6 0.6 0.6 1" />
-            </material>
-        </visual>
-        <!-- Hubcap -->
-        <visual>
-            <origin rpy="${pi/2} 0 0" xyz="0 -0.18 0" />
-            <geometry>
-                <box size="0.02 0.5 0.02" />
-            </geometry>
-            <material name="Grey">
-                <color rgba="0.6 0.6 0.6 1" />
+    <link name="rear_right_wheel_link">
+        <inertial>
+            <mass value="1" />
+            <origin xyz="0 0 0" rpy="0 0 0" />
+            <inertia ixx="0.002526666666667" ixy="0" ixz="0" iyy="0.002526666666667" iyz="0" izz="0.005"/>
+        </inertial>
+        <collision>
+            <origin xyz="0 0 0" rpy="0 0 0"/>
+            <geometry>
+                <mesh filename="package://isa_afa_3/meshes/wheel_right.stl" />
+            </geometry>
+        </collision>
+        <visual>
+            <origin xyz="0 0 0" rpy="0 0 0"/>
+            <geometry>
+                <mesh filename="package://isa_afa_3/meshes/wheel_right.stl" />
+            </geometry>
+            <material name="Black">
+                <color rgba="0.1 0.1 0.1 1" />
             </material>
         </visual>
     </link>
     <!-- Link - front left wheel -->
-    <link name="link_front_left_wheel">
-        <inertial>
-            <mass value="1" />
-            <origin xyz="0 0 0" rpy="0 0 0" />
-            <inertia ixx="0.002526666666667" ixy="0" ixz="0" iyy="0.002526666666667" iyz="0" izz="0.005"/>
-        </inertial>
-        <!-- Tires -->
-        <collision>
-            <origin rpy="${pi/2} 0 0" xyz="0 0.18 0" />
-            <geometry>
-                <cylinder length="0.12" radius="0.4"/>
-            </geometry>
-        </collision>
-        <visual>
-            <origin rpy="${pi/2} 0 0" xyz="0 0.18 0" />
-            <geometry>
-                <mesh filename="package://isa_afa_3/meshes/wheel.stl" />
-            </geometry>
-            <material name="Black">
-                <color rgba="0.1 0.1 0.1 1" />
-            </material>
-        </visual>
-        <!-- Axle -->
-        <collision>
-            <origin rpy="${pi/2} 0 0" xyz="0 0.06 0" />
-            <geometry>
-                <cylinder length="0.12" radius="0.08"/>
-            </geometry>
-        </collision>
-        <visual>
-            <origin rpy="${pi/2} 0 0" xyz="0 0.06 0" />
-            <geometry>
-                <cylinder length="0.12" radius="0.08"/>
-            </geometry>
-            <material name="Grey">
-                <color rgba="0.6 0.6 0.6 1" />
-            </material>
-        </visual>
-        <!-- Hubcap -->
-        <visual>
-            <origin rpy="${pi/2} 0 0" xyz="0 0.18 0" />
-            <geometry>
-                <box size="0.02 0.5 0.02" />
-            </geometry>
-            <material name="Grey">
-                <color rgba="0.6 0.6 0.6 1" />
+    <link name="front_left_wheel_link">
+        <inertial>
+            <mass value="1" />
+            <origin xyz="0 0 0" rpy="0 0 0" />
+            <inertia ixx="0.002526666666667" ixy="0" ixz="0" iyy="0.002526666666667" iyz="0" izz="0.005"/>
+        </inertial>
+        <collision>
+            <origin xyz="0 0 0" rpy="0 0 0"/>
+            <geometry>
+                <mesh filename="package://isa_afa_3/meshes/wheel_left.stl" />
+            </geometry>
+        </collision>
+        <visual>
+            <origin xyz="0 0 0" rpy="0 0 0"/>
+            <geometry>
+                <mesh filename="package://isa_afa_3/meshes/wheel_left.stl" />
+            </geometry>
+            <material name="Black">
+                <color rgba="0.1 0.1 0.1 1" />
             </material>
         </visual>
     </link>
     <!-- Link - front right wheel -->
-    <link name="link_front_right_wheel">
-        <inertial>
-            <mass value="1" />
-            <origin xyz="0 0 0" rpy="0 0 0" />
-            <inertia ixx="0.002526666666667" ixy="0" ixz="0" iyy="0.002526666666667" iyz="0" izz="0.005"/>
-        </inertial>
-        <!-- Tires -->
-        <collision>
-            <origin rpy="${pi/2} 0 0" xyz="0 -0.18 0" />
-            <geometry>
-                <cylinder length="0.12" radius="0.4"/>
-            </geometry>
-        </collision>
-        <visual>
-            <origin rpy="${pi/2} 0 0" xyz="0 -0.18 0" />
-            <geometry>
-                <mesh filename="package://isa_afa_3/meshes/wheel.stl" />
-            </geometry>
-            <material name="Black">
-                <color rgba="0.1 0.1 0.1 1" />
-            </material>
-        </visual>
-        <!-- Axle -->
-        <collision>
-            <origin rpy="${pi/2} 0 0" xyz="0 -0.06 0" />
-            <geometry>
-                <cylinder length="0.12" radius="0.08"/>
-            </geometry>
-        </collision>
-        <visual>
-            <origin rpy="${pi/2} 0 0" xyz="0 -0.06 0" />
-            <geometry>
-                <cylinder length="0.12" radius="0.08"/>
-            </geometry>
-            <material name="Grey">
-                <color rgba="0.6 0.6 0.6 1" />
-            </material>
-        </visual>
-        <!-- Hubcap -->
-        <visual>
-            <origin rpy="${pi/2} 0 0" xyz="0 -0.18 0" />
-            <geometry>
-                <box size="0.02 0.5 0.02" />
-            </geometry>
-            <material name="Grey">
-                <color rgba="0.6 0.6 0.6 1" />
+    <link name="front_right_wheel_link">
+        <inertial>
+            <mass value="1" />
+            <origin xyz="0 0 0" rpy="0 0 0" />
+            <inertia ixx="0.002526666666667" ixy="0" ixz="0" iyy="0.002526666666667" iyz="0" izz="0.005"/>
+        </inertial>
+        <collision>
+            <origin xyz="0 0 0" rpy="0 0 0"/>
+            <geometry>
+                <mesh filename="package://isa_afa_3/meshes/wheel_right.stl" />
+            </geometry>
+        </collision>
+        <visual>
+            <origin xyz="0 0 0" rpy="0 0 0"/>
+            <geometry>
+                <mesh filename="package://isa_afa_3/meshes/wheel_right.stl" />
+            </geometry>
+            <material name="Black">
+                <color rgba="0.1 0.1 0.1 1" />
+            </material>
+        </visual>
+    </link>
+    <!-- Link - front axle -->
+    <link name="front_axle_link">
+        <inertial>
+            <mass value="1" />
+            <origin xyz="0 0 0" rpy="0 0 0" />
+            <inertia ixx="0.002526666666667" ixy="0" ixz="0" iyy="0.002526666666667" iyz="0" izz="0.005"/>
+        </inertial>
+        <collision>
+            <origin rpy="${pi/2} 0 0" xyz="0 0 0"/>
+            <geometry>
+                <cylinder length="1.4" radius="0.1"/>
+            </geometry>
+        </collision>
+        <visual>
+            <origin rpy="${pi/2} 0 0" xyz="0 0 0"/>
+            <geometry>
+                <cylinder length="1.4" radius="0.1"/>
+            </geometry>
+            <material name="Black">
+                <color rgba="0.1 0.1 0.1 1" />
+            </material>
+        </visual>
+    </link>
+    <!-- Link - rear axle -->
+    <link name="rear_axle_link">
+        <inertial>
+            <mass value="1" />
+            <origin xyz="0 0 0" rpy="0 0 0" />
+            <inertia ixx="0.002526666666667" ixy="0" ixz="0" iyy="0.002526666666667" iyz="0" izz="0.005"/>
+        </inertial>
+        <collision>
+            <origin rpy="${pi/2} 0 0" xyz="0 0 0"/>
+            <geometry>
+                <cylinder length="1.4" radius="0.1"/>
+            </geometry>
+        </collision>
+        <visual>
+            <origin rpy="${pi/2} 0 0" xyz="0 0 0"/>
+            <geometry>
+                <cylinder length="1.4" radius="0.1"/>
+            </geometry>
+            <material name="Black">
+                <color rgba="0.1 0.1 0.1 1" />
             </material>
         </visual>
     </link>
     <!-- Link - left hinge -->
-    <link name="link_left_hinge">
+    <link name="left_hinge_link">
         <inertial>
             <mass value="0.001"/>
@@ -234,5 +182,5 @@
     </link>
     <!-- Link - right hinge -->
-    <link name="link_right_hinge">
+    <link name="right_hinge_link">
         <inertial>
             <mass value="0.001"/>
@@ -241,60 +189,75 @@
     </link>
     <!-- JOINTS -->
-    <!-- Joint - chassis / rear left wheel -->
-    <joint name="joint_chassis_rear_left_wheel" type="continuous">
-        <origin rpy="0 0 0" xyz="-0.5 0.65 0" />
-        <child link="link_rear_left_wheel" />
-        <parent link="link_chassis" />
-        <axis rpy="0 0 0" xyz="0 1 0" />
-        <limit effort="10000" velocity="1000" />
+    <!-- Joint - chassis / front axle -->
+    <joint name="chassis_front_axle_joint" type="fixed">
+        <origin rpy="0 0 0" xyz="0 0 0" />
+        <child link="front_axle_link" />
+        <parent link="base_link" />
         <joint_properties damping="1.0" friction="1.0" />
     </joint>
-    <!-- Joint - chassis / rear right wheel -->
-    <joint name="joint_chassis_rear_right_wheel" type="continuous">
-        <origin rpy="0 0 0" xyz="-0.5 -0.65 0" />
-        <child link="link_rear_right_wheel" />
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