Commit message: chore: format

File: src/isa_afa_3/src/description/robot.xacro (robot description, xacro)
@@ -1,282 +1,282 @@
-<?xml version="1.0"?>
-<robot name="robot" xmlns:xacro="http://www.ros.org/wiki/xacro">
-	<xacro:include filename="$(find isa_afa_3)/src/description/robot.gazebo" />
-	<!-- Parameters -->
-	<xacro:property name="chassis_mass" value="1500" />
-	<xacro:property name="chassis_length" value="4.5" />
-	<xacro:property name="chassis_width" value="1.8" />
-	<xacro:property name="chassis_height" value="1.4" />
-	<xacro:property name="axle_mass" value="50" />
-	<xacro:property name="axle_radius" value="0.1" />
-	<xacro:property name="axle_width" value="1.4" />
-	<xacro:property name="wheel_mass" value="20" />
-	<xacro:property name="wheel_radius" value="0.3" />
-	<xacro:property name="wheel_width" value="0.2" />
-	<xacro:property name="wheel_base" value="2.6" />
-	<xacro:property name="lidar_mass" value="0.5" />
-	<xacro:property name="lidar_radius" value="0.15" />
-	<xacro:property name="lidar_length" value="0.2" />
-	<!-- Commonly used inertial: Box  -->
-	<xacro:macro name="box_inertia" params="m w h d">
-		<inertial>
-			<origin xyz="0 0 0" rpy="${pi/2} 0 ${pi/2}" />
-			<mass value="${m}" />
-			<inertia ixx="${(m/12) * (h*h + d*d)}" ixy="0.0" ixz="0.0" iyy="${(m/12) * (w*w + d*d)}" iyz="0.0" izz="${(m/12) * (w*w + h*h)}" />
-		</inertial>
-	</xacro:macro>
-	<!-- Commonly used inertial: Cylinder  -->
-	<xacro:macro name="cylinder_inertia" params="m r h">
-		<inertial>
-			<origin xyz="0 0 0" rpy="${pi/2} 0 0" />
-			<mass value="${m}" />
-			<inertia ixx="${(m/12) * (3*r*r + h*h)}" ixy="0.0" ixz="0.0" iyy="${(m/12) * (3*r*r + h*h)}" iyz="0.0" izz="${(m/2) * (r*r)}" />
-		</inertial>
-	</xacro:macro>
-	<!-- Link - chassis -->
-	<link name="base_link">
-		<xacro:box_inertia m="${chassis_mass}" w="${chassis_width}" d="${chassis_length}" h="${chassis_height}"/>
-		<collision>
-			<origin xyz="0 0 0" rpy="0 0 0"/>
-			<geometry>
-				<mesh filename="package://isa_afa_3/meshes/chassis.stl"/>
-			</geometry>
-		</collision>
-		<visual>
-			<origin xyz="0 0 0" rpy="0 0 0"/>
-			<geometry>
-				<mesh filename="package://isa_afa_3/meshes/chassis.stl"/>
-			</geometry>
-			<material name="DarkBlue">
-				<color rgba="0.2 0.2 0.4 1" />
-			</material>
-		</visual>
-	</link>
-	<!-- Link - robot footprint -->
-	<link name='base_footprint'>
-		<inertial>
-			<mass value="0.01" />
-			<inertia ixx="0.001" ixy="0.0" ixz="0.0" iyy="0.001" iyz="0.0" izz="0.001" />
-		</inertial>
-	</link>
-	<!-- Link - rear left wheel -->
-	<link name="rear_left_wheel_link">
-		<xacro:cylinder_inertia m="${wheel_mass}" r="${wheel_radius}" h="${wheel_width}"/>
-		<collision>
-			<origin xyz="0 0 0" rpy="0 0 0"/>
-			<geometry>
-				<mesh filename="package://isa_afa_3/meshes/wheel_left.stl" />
-			</geometry>
-		</collision>
-		<visual>
-			<origin xyz="0 0 0" rpy="0 0 0"/>
-			<geometry>
-				<mesh filename="package://isa_afa_3/meshes/wheel_left.stl" />
-			</geometry>
-			<material name="Black">
-				<color rgba="0.1 0.1 0.1 1" />
-			</material>
-		</visual>
-	</link>
-	<!-- Link - rear right wheel -->
-	<link name="rear_right_wheel_link">
-		<xacro:cylinder_inertia m="${wheel_mass}" r="${wheel_radius}" h="${wheel_width}"/>
-		<collision>
-			<origin xyz="0 0 0" rpy="0 0 0"/>
-			<geometry>
-				<mesh filename="package://isa_afa_3/meshes/wheel_right.stl" />
-			</geometry>
-		</collision>
-		<visual>
-			<origin xyz="0 0 0" rpy="0 0 0"/>
-			<geometry>
-				<mesh filename="package://isa_afa_3/meshes/wheel_right.stl" />
-			</geometry>
-			<material name="Black">
-				<color rgba="0.1 0.1 0.1 1" />
-			</material>
-		</visual>
-	</link>
-	<!-- Link - front left wheel -->
-	<link name="front_left_wheel_link">
-		<xacro:cylinder_inertia m="${wheel_mass}" r="${wheel_radius}" h="${wheel_width}"/>
-		<collision>
-			<origin xyz="0 0 0" rpy="0 0 0"/>
-			<geometry>
-				<mesh filename="package://isa_afa_3/meshes/wheel_left.stl" />
-			</geometry>
-		</collision>
-		<visual>
-			<origin xyz="0 0 0" rpy="0 0 0"/>
-			<geometry>
-				<mesh filename="package://isa_afa_3/meshes/wheel_left.stl" />
-			</geometry>
-			<material name="Black">
-				<color rgba="0.1 0.1 0.1 1" />
-			</material>
-		</visual>
-	</link>
-	<!-- Link - front right wheel -->
-	<link name="front_right_wheel_link">
-		<xacro:cylinder_inertia m="${wheel_mass}" r="${wheel_radius}" h="${wheel_width}"/>
-		<collision>
-			<origin xyz="0 0 0" rpy="0 0 0"/>
-			<geometry>
-				<mesh filename="package://isa_afa_3/meshes/wheel_right.stl" />
-			</geometry>
-		</collision>
-		<visual>
-			<origin xyz="0 0 0" rpy="0 0 0"/>
-			<geometry>
-				<mesh filename="package://isa_afa_3/meshes/wheel_right.stl" />
-			</geometry>
-			<material name="Black">
-				<color rgba="0.1 0.1 0.1 1" />
-			</material>
-		</visual>
-	</link>
-	<!-- Link - front axle -->
-	<link name="front_axle_link">
-		<xacro:cylinder_inertia m="${axle_mass}" r="${axle_radius}" h="${axle_width}"/>
-		<collision>
-			<origin rpy="${pi/2} 0 0" xyz="0 0 0"/>
-			<geometry>
-				<cylinder length="${axle_width}" radius="${axle_radius}"/>
-			</geometry>
-		</collision>
-		<visual>
-			<origin rpy="${pi/2} 0 0" xyz="0 0 0"/>
-			<geometry>
-				<cylinder length="${axle_width}" radius="${axle_radius}"/>
-			</geometry>
-			<material name="Black">
-				<color rgba="0.1 0.1 0.1 1" />
-			</material>
-		</visual>
-	</link>
-	<!-- Link - rear axle -->
-	<link name="rear_axle_link">
-		<xacro:cylinder_inertia m="${axle_mass}" r="${axle_radius}" h="${axle_width}"/>
-		<collision>
-			<origin rpy="${pi/2} 0 0" xyz="0 0 0"/>
-			<geometry>
-				<cylinder length="${axle_width}" radius="${axle_radius}"/>
-			</geometry>
-		</collision>
-		<visual>
-			<origin rpy="${pi/2} 0 0" xyz="0 0 0"/>
-			<geometry>
-				<cylinder length="${axle_width}" radius="${axle_radius}"/>
-			</geometry>
-			<material name="Black">
-				<color rgba="0.1 0.1 0.1 1" />
-			</material>
-		</visual>
-	</link>
-	<!-- Link - left hinge -->
-	<link name="left_hinge_link">
-		<inertial>
-			<mass value="0.01"/>
-			<inertia ixx="0.001" ixy = "0" ixz = "0" iyy="0.001" iyz = "0" izz="0.001"/>
-		</inertial>
-	</link>
-	<!-- Link - right hinge -->
-	<link name="right_hinge_link">
-		<inertial>
-			<mass value="0.01"/>
-			<inertia ixx="0.001" ixy = "0" ixz = "0" iyy="0.001" iyz = "0" izz="0.001"/>
-		</inertial>
-	</link>
-	<link name="lidar_link">
-		<inertial>
-			<origin xyz="0 0 0" rpy="0 0 0" />
-			<mass value="${lidar_mass}" />
-			<inertia ixx="0.00025267" ixy="0" ixz="0" iyy="0.00025267" iyz="0" izz="0.0005"/>
-		</inertial>
-		<visual>
-			<origin xyz="0 0 0" rpy="0 0 0" />
-			<geometry>
-				<cylinder radius="${lidar_radius}" length="${lidar_length}"/>
-			</geometry>
-			<material name="Red">
-				<color rgba="0.7 0.1 0.1 1" />
-			</material>
-		</visual>
-		<collision>
-			<origin xyz="0 0 0" rpy="0 0 0"/>
-			<geometry>
-				<cylinder radius="${lidar_radius}" length="${lidar_length}"/>
-			</geometry>
-		</collision>
-	</link>
-		<!-- Joint - chassis / footprint -->
-	<joint name='base_joint' type='fixed'>
-		<origin rpy="0 0 0" xyz="0 0 -${wheel_radius}" />
-		<child link="base_footprint" />
-		<parent link="base_link" />
-	</joint>
-	<!-- Joint - chassis / front axle -->
-	<joint name="chassis_front_axle_joint" type="fixed">
-		<origin rpy="0 0 0" xyz="0 0 0" />
-		<child link="front_axle_link" />
-		<parent link="base_link" />
-		<joint_properties damping="1.0" friction="1.0" />
-	</joint>
-	<!-- Joint - chassis / rear axle -->
-	<joint name="chassis_rear_axle_joint" type="fixed">
-		<origin rpy="0 0 0" xyz="-${wheel_base} 0 0" />
-		<child link="rear_axle_link" />
-		<parent link="base_link" />
-		<joint_properties damping="1.0" friction="1.0" />
-	</joint>
-	<!-- Joint - front axle / left hinge -->
-	<joint name="steering_left_hinge_joint" type="revolute">
-		<child link="left_hinge_link" />
-		<parent link="front_axle_link" />
-		<origin xyz="0 ${axle_width/2} 0" rpy="0 0 0" />
-		<axis xyz="0 0 1" />
-		<limit lower="-0.7" upper="0.7" effort="10" velocity="100" />
-	</joint>
-	<!-- Joint - front axle / right hinge -->
-	<joint name="steering_right_hinge_joint" type="revolute">
-		<child link="right_hinge_link" />
-		<parent link="front_axle_link" />
-		<origin xyz="0 -${axle_width/2} 0" rpy="0 0 0" />
-		<axis xyz="0 0 1" />
-		<limit lower="-0.7" upper="0.7" effort="10" velocity="100" />
-	</joint>
-	<!-- Joint - left hinge / front left wheel -->
-	<joint name="left_hinge_wheel_joint" type="continuous">
-		<child link="front_left_wheel_link" />
-		<parent link="left_hinge_link" />
-		<origin xyz="0 0 0" rpy="0 0 0" />
-		<axis xyz="0 1 0" />
-	</joint>
-	<!-- Joint - right hinge / front right wheel -->
-	<joint name="right_hinge_wheel_joint" type="continuous">
-		<child link="front_right_wheel_link" />
-		<parent link="right_hinge_link" />
-		<origin xyz="0 0 0" rpy="0 0 0" />
-		<axis xyz="0 1 0" />
-	</joint>
-	<!-- Joint - rear axle / rear left wheel -->
-	<joint name="rear_axle_left_wheel_joint" type="continuous">
-		<child link="rear_left_wheel_link" />
-		<parent link="rear_axle_link" />
-		<origin xyz="0 ${axle_width/2} 0" rpy="0 0 0" />
-		<axis xyz="0 1 0" />
-	</joint>
-	<!-- Joint - rear axle / rear right wheel -->
-	<joint name="rear_axle_right_wheel_joint" type="continuous">
-		<child link="rear_right_wheel_link" />
-		<parent link="rear_axle_link" />
-		<origin xyz="0 -${axle_width/2} 0" rpy="0 0 0" />
-		<axis xyz="0 1 0" />
-	</joint>
-	<!-- Laser scan -->
-	<joint name="lidar_joint" type="fixed">
-		<origin rpy="0 0 0" xyz="-${wheel_base/2} 0 ${lidar_length/2+chassis_height}" />
-		<child link="lidar_link" />
-		<parent link="base_link" />
-		<joint_properties damping="1.0" friction="1.0" />
-	</joint>
+<?xml version="1.0" encoding="UTF-8"?>
+<robot xmlns:xacro="http://www.ros.org/wiki/xacro" name="robot">
+  <xacro:include filename="$(find isa_afa_3)/src/description/robot.gazebo" />
+  <!-- Parameters -->
+  <xacro:property name="chassis_mass" value="1500" />
+  <xacro:property name="chassis_length" value="4.5" />
+  <xacro:property name="chassis_width" value="1.8" />
+  <xacro:property name="chassis_height" value="1.4" />
+  <xacro:property name="axle_mass" value="50" />
+  <xacro:property name="axle_radius" value="0.1" />
+  <xacro:property name="axle_width" value="1.4" />
+  <xacro:property name="wheel_mass" value="20" />
+  <xacro:property name="wheel_radius" value="0.3" />
+  <xacro:property name="wheel_width" value="0.2" />
+  <xacro:property name="wheel_base" value="2.6" />
+  <xacro:property name="lidar_mass" value="0.5" />
+  <xacro:property name="lidar_radius" value="0.15" />
+  <xacro:property name="lidar_length" value="0.2" />
+  <!-- Commonly used inertial: Box  -->
+  <xacro:macro name="box_inertia" params="m w h d">
+    <inertial>
+      <origin xyz="0 0 0" rpy="${pi/2} 0 ${pi/2}" />
+      <mass value="${m}" />
+      <inertia ixx="${(m/12) * (h*h + d*d)}" ixy="0.0" ixz="0.0" iyy="${(m/12) * (w*w + d*d)}" iyz="0.0" izz="${(m/12) * (w*w + h*h)}" />
+    </inertial>
+  </xacro:macro>
+  <!-- Commonly used inertial: Cylinder  -->
+  <xacro:macro name="cylinder_inertia" params="m r h">
+    <inertial>
+      <origin xyz="0 0 0" rpy="${pi/2} 0 0" />
+      <mass value="${m}" />
+      <inertia ixx="${(m/12) * (3*r*r + h*h)}" ixy="0.0" ixz="0.0" iyy="${(m/12) * (3*r*r + h*h)}" iyz="0.0" izz="${(m/2) * (r*r)}" />
+    </inertial>
+  </xacro:macro>
+  <!-- Link - chassis -->
+  <link name="base_link">
+    <xacro:box_inertia m="${chassis_mass}" w="${chassis_width}" d="${chassis_length}" h="${chassis_height}" />
+    <collision>
+      <origin xyz="0 0 0" rpy="0 0 0" />
+      <geometry>
+        <mesh filename="package://isa_afa_3/meshes/chassis.stl" />
+      </geometry>
+    </collision>
+    <visual>
+      <origin xyz="0 0 0" rpy="0 0 0" />
+      <geometry>
+        <mesh filename="package://isa_afa_3/meshes/chassis.stl" />
+      </geometry>
+      <material name="DarkBlue">
+        <color rgba="0.2 0.2 0.4 1" />
+      </material>
+    </visual>
+  </link>
+  <!-- Link - robot footprint -->
+  <link name="base_footprint">
+    <inertial>
+      <mass value="0.01" />
+      <inertia ixx="0.001" ixy="0.0" ixz="0.0" iyy="0.001" iyz="0.0" izz="0.001" />
+    </inertial>
+  </link>
+  <!-- Link - rear left wheel -->
+  <link name="rear_left_wheel_link">
+    <xacro:cylinder_inertia m="${wheel_mass}" r="${wheel_radius}" h="${wheel_width}" />
+    <collision>
+      <origin xyz="0 0 0" rpy="0 0 0" />
+      <geometry>
+        <mesh filename="package://isa_afa_3/meshes/wheel_left.stl" />
+      </geometry>
+    </collision>
+    <visual>
+      <origin xyz="0 0 0" rpy="0 0 0" />
+      <geometry>
+        <mesh filename="package://isa_afa_3/meshes/wheel_left.stl" />
+      </geometry>
+      <material name="Black">
+        <color rgba="0.1 0.1 0.1 1" />
+      </material>
+    </visual>
+  </link>
+  <!-- Link - rear right wheel -->
+  <link name="rear_right_wheel_link">
+    <xacro:cylinder_inertia m="${wheel_mass}" r="${wheel_radius}" h="${wheel_width}" />
+    <collision>
+      <origin xyz="0 0 0" rpy="0 0 0" />
+      <geometry>
+        <mesh filename="package://isa_afa_3/meshes/wheel_right.stl" />
+      </geometry>
+    </collision>
+    <visual>
+      <origin xyz="0 0 0" rpy="0 0 0" />
+      <geometry>
+        <mesh filename="package://isa_afa_3/meshes/wheel_right.stl" />
+      </geometry>
+      <material name="Black">
+        <color rgba="0.1 0.1 0.1 1" />
+      </material>
+    </visual>
+  </link>
+  <!-- Link - front left wheel -->
+  <link name="front_left_wheel_link">
+    <xacro:cylinder_inertia m="${wheel_mass}" r="${wheel_radius}" h="${wheel_width}" />
+    <collision>
+      <origin xyz="0 0 0" rpy="0 0 0" />
+      <geometry>
+        <mesh filename="package://isa_afa_3/meshes/wheel_left.stl" />
+      </geometry>
+    </collision>
+    <visual>
+      <origin xyz="0 0 0" rpy="0 0 0" />
+      <geometry>
+        <mesh filename="package://isa_afa_3/meshes/wheel_left.stl" />
+      </geometry>
+      <material name="Black">
+        <color rgba="0.1 0.1 0.1 1" />
+      </material>
+    </visual>
+  </link>
+  <!-- Link - front right wheel -->
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
Commit message: feat: add imu and camera

File: src/isa_afa_3/src/description/robot.xacro (robot description, xacro)
@@ -3,5 +3,6 @@
   <xacro:include filename="$(find isa_afa_3)/src/description/robot.gazebo" />
   <!-- Parameters -->
-  <xacro:property name="chassis_mass" value="1500" />
+  <!-- <xacro:property name="chassis_mass" value="1500" /> -->
+  <xacro:property name="chassis_mass" value="50" />
   <xacro:property name="chassis_length" value="4.5" />
   <xacro:property name="chassis_width" value="1.8" />
@@ -17,4 +18,8 @@
   <xacro:property name="lidar_radius" value="0.15" />
   <xacro:property name="lidar_length" value="0.2" />
+  <xacro:property name="camera_mass" value="0.05" />
+  <xacro:property name="camera_width" value="0.1" />
+  <xacro:property name="camera_depth" value="0.03" />
+  <xacro:property name="camera_height" value="0.07" />
   <!-- Commonly used inertial: Box  -->
   <xacro:macro name="box_inertia" params="m w h d">
@@ -187,4 +192,5 @@
     </inertial>
   </link>
+  <!-- Link - lidar -->
   <link name="lidar_link">
     <inertial>
@@ -206,4 +212,36 @@
       <geometry>
         <cylinder radius="${lidar_radius}" length="${lidar_length}" />
+      </geometry>
+    </collision>
+  </link>
+  <!-- Link - imu -->
+  <link name="imu_link">
+    <xacro:box_inertia m="0.1" w="0.1" d="0.1" h="0.1"/>
+    <visual>
+      <origin xyz="0 0 0" rpy="0 0 0" />
+      <geometry>
+        <box size="0.1 0.1 0.1" />
+      </geometry>
+    </visual>
+    <collision>
+      <origin xyz="0 0 0" rpy="0 0 0" />
+      <geometry>
+        <box size="0.1 0.1 0.1" />
+      </geometry>
+    </collision>
+  </link>
+  <!-- Link - camera -->
+  <link name="camera_link">
+    <xacro:box_inertia m="${camera_mass}" w="${camera_width}" d="${camera_depth}" h="${camera_height}"/>
+    <visual>
+      <origin xyz="0 0 0" rpy="0 0 0" />
+      <geometry>
+        <box size="0.1 0.1 0.1" />
+      </geometry>
+    </visual>
+    <collision>
+      <origin xyz="0 0 0" rpy="0 0 0" />
+      <geometry>
+        <box size="0.1 0.1 0.1" />
       </geometry>
     </collision>
@@ -273,5 +311,5 @@
     <axis xyz="0 1 0" />
   </joint>
-  <!-- Laser scan -->
+  <!-- Joint - chassis / lidar -->
   <joint name="lidar_joint" type="fixed">
     <origin rpy="0 0 0" xyz="-${wheel_base/2} 0 ${lidar_length/2+chassis_height}" />
@@ -280,3 +318,14 @@
     <joint_properties damping="1.0" friction="1.0" />
   </joint>
+  <!-- Joint - chassis / imu -->
+  <joint name='imu_joint' type='fixed'>
+    <child link="imu_link" />
+    <parent link="base_link" />
+  </joint>
+  <!-- Joint - chassis / camera -->
+  <joint name='camera_joint' type='fixed'>
+    <origin rpy="0 0 0" xyz="0.9 0 0.3" />
+    <child link="camera_link" />
+    <parent link="base_link" />
+  </joint>
 </robot>
