Commit message: feat: optimizations for ackermann plugin

File: src/isa_afa_3/src/description/robot.xacro (robot description, xacro)
@@ -2,7 +2,6 @@
 <robot xmlns:xacro="http://www.ros.org/wiki/xacro" name="robot">
   <xacro:include filename="$(find isa_afa_3)/src/description/robot.gazebo" />
-  <!-- Parameters -->
-  <!-- <xacro:property name="chassis_mass" value="1500" /> -->
-  <xacro:property name="chassis_mass" value="50" />
+  <!-- Properties -->
+  <xacro:property name="chassis_mass" value="1000" />
   <xacro:property name="chassis_length" value="4.5" />
   <xacro:property name="chassis_width" value="1.8" />
@@ -10,7 +9,7 @@
   <xacro:property name="axle_mass" value="50" />
   <xacro:property name="axle_radius" value="0.1" />
-  <xacro:property name="axle_width" value="1.4" />
+  <xacro:property name="axle_width" value="1.0" />
   <xacro:property name="wheel_mass" value="20" />
-  <xacro:property name="wheel_radius" value="0.3" />
+  <xacro:property name="wheel_radius" value="0.27" />
   <xacro:property name="wheel_width" value="0.2" />
   <xacro:property name="wheel_base" value="2.6" />
@@ -23,7 +22,7 @@
   <xacro:property name="camera_height" value="0.07" />
   <!-- Commonly used inertial: Box  -->
-  <xacro:macro name="box_inertia" params="m w h d">
-    <inertial>
-      <origin xyz="0 0 0" rpy="${pi/2} 0 ${pi/2}" />
+  <xacro:macro name="box_inertia" params="m w h d x y z">
+    <inertial>
+      <origin xyz="${x} ${y} ${z}" rpy="${pi/2} 0 ${pi/2}" />
       <mass value="${m}" />
       <inertia ixx="${(m/12) * (h*h + d*d)}" ixy="0.0" ixz="0.0" iyy="${(m/12) * (w*w + d*d)}" iyz="0.0" izz="${(m/12) * (w*w + h*h)}" />
@@ -40,5 +39,5 @@
   <!-- Link - chassis -->
   <link name="base_link">
-    <xacro:box_inertia m="${chassis_mass}" w="${chassis_width}" d="${chassis_length}" h="${chassis_height}" />
+    <xacro:box_inertia m="${chassis_mass}" w="${chassis_width}" d="${chassis_length}" h="${chassis_height}" x="-${chassis_length/2-0.9}" y="0" z="${chassis_height/2}" />
     <collision>
       <origin xyz="0 0 0" rpy="0 0 0" />
@@ -68,13 +67,13 @@
     <xacro:cylinder_inertia m="${wheel_mass}" r="${wheel_radius}" h="${wheel_width}" />
     <collision>
-      <origin xyz="0 0 0" rpy="0 0 0" />
-      <geometry>
-        <mesh filename="package://isa_afa_3/meshes/wheel_left.stl" />
-      </geometry>
-    </collision>
-    <visual>
-      <origin xyz="0 0 0" rpy="0 0 0" />
-      <geometry>
-        <mesh filename="package://isa_afa_3/meshes/wheel_left.stl" />
+      <origin rpy="${pi/2} 0 0" xyz="0 0 0" />
+      <geometry>
+        <cylinder length="${wheel_width}" radius="${wheel_radius}" />
+      </geometry>
+    </collision>
+    <visual>
+      <origin rpy="${pi/2} 0 0" xyz="0 0 0" />
+      <geometry>
+        <cylinder length="${wheel_width}" radius="${wheel_radius}" />
       </geometry>
       <material name="Black">
@@ -87,13 +86,13 @@
     <xacro:cylinder_inertia m="${wheel_mass}" r="${wheel_radius}" h="${wheel_width}" />
     <collision>
-      <origin xyz="0 0 0" rpy="0 0 0" />
-      <geometry>
-        <mesh filename="package://isa_afa_3/meshes/wheel_right.stl" />
-      </geometry>
-    </collision>
-    <visual>
-      <origin xyz="0 0 0" rpy="0 0 0" />
-      <geometry>
-        <mesh filename="package://isa_afa_3/meshes/wheel_right.stl" />
+      <origin rpy="${pi/2} 0 0" xyz="0 0 0" />
+      <geometry>
+        <cylinder length="${wheel_width}" radius="${wheel_radius}" />
+      </geometry>
+    </collision>
+    <visual>
+      <origin rpy="${pi/2} 0 0" xyz="0 0 0" />
+      <geometry>
+        <cylinder length="${wheel_width}" radius="${wheel_radius}" />
       </geometry>
       <material name="Black">
@@ -106,13 +105,13 @@
     <xacro:cylinder_inertia m="${wheel_mass}" r="${wheel_radius}" h="${wheel_width}" />
     <collision>
-      <origin xyz="0 0 0" rpy="0 0 0" />
-      <geometry>
-        <mesh filename="package://isa_afa_3/meshes/wheel_left.stl" />
-      </geometry>
-    </collision>
-    <visual>
-      <origin xyz="0 0 0" rpy="0 0 0" />
-      <geometry>
-        <mesh filename="package://isa_afa_3/meshes/wheel_left.stl" />
+      <origin rpy="${pi/2} 0 0" xyz="0 0 0" />
+      <geometry>
+        <cylinder length="${wheel_width}" radius="${wheel_radius}" />
+      </geometry>
+    </collision>
+    <visual>
+      <origin rpy="${pi/2} 0 0" xyz="0 0 0" />
+      <geometry>
+        <cylinder length="${wheel_width}" radius="${wheel_radius}" />
       </geometry>
       <material name="Black">
@@ -125,13 +124,13 @@
     <xacro:cylinder_inertia m="${wheel_mass}" r="${wheel_radius}" h="${wheel_width}" />
     <collision>
-      <origin xyz="0 0 0" rpy="0 0 0" />
-      <geometry>
-        <mesh filename="package://isa_afa_3/meshes/wheel_right.stl" />
-      </geometry>
-    </collision>
-    <visual>
-      <origin xyz="0 0 0" rpy="0 0 0" />
-      <geometry>
-        <mesh filename="package://isa_afa_3/meshes/wheel_right.stl" />
+      <origin rpy="${pi/2} 0 0" xyz="0 0 0" />
+      <geometry>
+        <cylinder length="${wheel_width}" radius="${wheel_radius}" />
+      </geometry>
+    </collision>
+    <visual>
+      <origin rpy="${pi/2} 0 0" xyz="0 0 0" />
+      <geometry>
+        <cylinder length="${wheel_width}" radius="${wheel_radius}" />
       </geometry>
       <material name="Black">
@@ -178,6 +177,6 @@
     </visual>
   </link>
-  <!-- Link - left hinge -->
-  <link name="left_hinge_link">
+  <!-- Link - left kingpin -->
+  <link name="left_kingpin_link">
     <inertial>
       <mass value="0.01" />
@@ -185,6 +184,6 @@
     </inertial>
   </link>
-  <!-- Link - right hinge -->
-  <link name="right_hinge_link">
+  <!-- Link - right kingpin -->
+  <link name="right_kingpin_link">
     <inertial>
       <mass value="0.01" />
@@ -217,5 +216,5 @@
   <!-- Link - imu -->
   <link name="imu_link">
-    <xacro:box_inertia m="0.1" w="0.1" d="0.1" h="0.1"/>
+    <xacro:box_inertia m="0.1" w="0.1" d="0.1" h="0.1" x="0" y="0" z="0" />
     <visual>
       <origin xyz="0 0 0" rpy="0 0 0" />
@@ -233,5 +232,5 @@
   <!-- Link - camera -->
   <link name="camera_link">
-    <xacro:box_inertia m="${camera_mass}" w="${camera_width}" d="${camera_depth}" h="${camera_height}"/>
+    <xacro:box_inertia m="${camera_mass}" w="${camera_width}" d="${camera_depth}" h="${camera_height}" x="0" y="0" z="0" />
     <visual>
       <origin xyz="0 0 0" rpy="0 0 0" />
@@ -258,5 +257,4 @@
     <child link="front_axle_link" />
     <parent link="base_link" />
-    <joint_properties damping="1.0" friction="1.0" />
   </joint>
   <!-- Joint - chassis / rear axle -->
@@ -265,34 +263,33 @@
     <child link="rear_axle_link" />
     <parent link="base_link" />
-    <joint_properties damping="1.0" friction="1.0" />
-  </joint>
-  <!-- Joint - front axle / left hinge -->
-  <joint name="steering_left_hinge_joint" type="revolute">
-    <child link="left_hinge_link" />
+  </joint>
+  <!-- Joint - front axle / left kingpin -->
+  <joint name="steering_left_kingpin_joint" type="revolute">
+    <child link="left_kingpin_link" />
     <parent link="front_axle_link" />
-    <origin xyz="0 ${axle_width/2} 0" rpy="0 0 0" />
+    <origin xyz="0 ${chassis_width/2-wheel_width} 0" rpy="0 0 0" />
     <axis xyz="0 0 1" />
-    <limit lower="-0.7" upper="0.7" effort="10" velocity="100" />
-  </joint>
-  <!-- Joint - front axle / right hinge -->
-  <joint name="steering_right_hinge_joint" type="revolute">
-    <child link="right_hinge_link" />
+    <limit lower="-0.7" upper="0.7" effort="100" velocity="1" />
+  </joint>
+  <!-- Joint - front axle / right kingpin -->
+  <joint name="steering_right_kingpin_joint" type="revolute">
+    <child link="right_kingpin_link" />
     <parent link="front_axle_link" />
-    <origin xyz="0 -${axle_width/2} 0" rpy="0 0 0" />
+    <origin xyz="0 -${chassis_width/2-wheel_width} 0" rpy="0 0 0" />
     <axis xyz="0 0 1" />
-    <limit lower="-0.7" upper="0.7" effort="10" velocity="100" />
-  </joint>
-  <!-- Joint - left hinge / front left wheel -->
-  <joint name="left_hinge_wheel_joint" type="continuous">
+    <limit lower="-0.7" upper="0.7" effort="100" velocity="1" />
+  </joint>
+  <!-- Joint - left kingpin / front left wheel -->
+  <joint name="left_kingpin_wheel_joint" type="continuous">
     <child link="front_left_wheel_link" />
-    <parent link="left_hinge_link" />
-    <origin xyz="0 0 0" rpy="0 0 0" />
+    <parent link="left_kingpin_link" />
+    <origin xyz="0 ${wheel_width/2} 0" rpy="0 0 0" />
     <axis xyz="0 1 0" />
   </joint>
-  <!-- Joint - right hinge / front right wheel -->
-  <joint name="right_hinge_wheel_joint" type="continuous">
+  <!-- Joint - right kingpin / front right wheel -->
+  <joint name="right_kingpin_wheel_joint" type="continuous">
     <child link="front_right_wheel_link" />
-    <parent link="right_hinge_link" />
-    <origin xyz="0 0 0" rpy="0 0 0" />
+    <parent link="right_kingpin_link" />
+    <origin xyz="0 -${wheel_width/2} 0" rpy="0 0 0" />
     <axis xyz="0 1 0" />
   </joint>
@@ -301,5 +298,5 @@
     <child link="rear_left_wheel_link" />
     <parent link="rear_axle_link" />
-    <origin xyz="0 ${axle_width/2} 0" rpy="0 0 0" />
+    <origin xyz="0 ${chassis_width/2-wheel_width/2} 0" rpy="0 0 0" />
     <axis xyz="0 1 0" />
   </joint>
@@ -308,5 +305,5 @@
     <child link="rear_right_wheel_link" />
     <parent link="rear_axle_link" />
-    <origin xyz="0 -${axle_width/2} 0" rpy="0 0 0" />
+    <origin xyz="0 -${chassis_width/2-wheel_width/2} 0" rpy="0 0 0" />
     <axis xyz="0 1 0" />
   </joint>
@@ -316,5 +313,4 @@
     <child link="lidar_link" />
     <parent link="base_link" />
-    <joint_properties damping="1.0" friction="1.0" />
   </joint>
   <!-- Joint - chassis / imu -->
